File: PowerMgmt.sch (KiCad schematic (older format))
At the start: 14 parts, among them J2 BATT_CONN, P1 USB_OTG, Q1 Q_NMOS_GSD, Q2 Q_PMOS_GSD, U4 AP2204K-3.0, U5 MCP73811T-420I-OT

Commit message: update schematics
Parts:
- P1: footprint Connect:USB_Micro-B -> Connectors_USB:USB_Micro-B_Molex_47346-0001
Connections:
- net labels added: VBUS
Changed lines of the file:
@@
 $EndComp
 $Comp
-L GND #PWR012
+L GND #PWR013
 U 1 1 59568C2C
 P 6700 3750
-F 0 "#PWR012" H 6700 3500 50  0001 C CNN
+F 0 "#PWR013" H 6700 3500 50  0001 C CNN
 F 1 "GND" H 6700 3600 50  0000 C CNN
 F 2 "" H 6700 3750 50  0000 C CNN
@@
 $EndComp
 $Comp
-L VDD #PWR013
+L VDD #PWR014
 U 1 1 59568C2F
 P 7100 2900
-F 0 "#PWR013" H 7100 2750 50  0001 C CNN
+F 0 "#PWR014" H 7100 2750 50  0001 C CNN
 F 1 "VDD" H 7100 3050 50  0000 C CNN
 F 2 "" H 7100 2900 50  0000 C CNN
@@
 $EndComp
 $Comp
-L GND #PWR014
+L GND #PWR015
 U 1 1 59568C3A
 P 3500 5100
-F 0 "#PWR014" H 3500 4850 50  0001 C CNN
+F 0 "#PWR015" H 3500 4850 50  0001 C CNN
 F 1 "GND" H 3500 4950 50  0000 C CNN
 F 2 "" H 3500 5100 50  0000 C CNN
@@
 $EndComp
 $Comp
-L +BATT #PWR015
+L +BATT #PWR016
 U 1 1 59568C5B
 P 3500 4900
-F 0 "#PWR015" H 3500 4750 50  0001 C CNN
+F 0 "#PWR016" H 3500 4750 50  0001 C CNN
 F 1 "+BATT" H 3500 5040 50  0000 C CNN
 F 2 "" H 3500 4900 50  0000 C CNN
@@
 Connection ~ 6700 3650
 $Comp
-L +BATT #PWR016
+L +BATT #PWR017
 U 1 1 5979B653
 P 4750 2900
-F 0 "#PWR016" H 4750 2750 50  0001 C CNN
+F 0 "#PWR017" H 4750 2750 50  0001 C CNN
 F 1 "+BATT" H 4750 3040 50  0000 C CNN
 F 2 "" H 4750 2900 50  0000 C CNN
@@
 $EndComp
 $Comp
-L GND #PWR017
+L GND #PWR018
 U 1 1 59D3742E
 P 3150 3650
-F 0 "#PWR017" H 3150 3400 50  0001 C CNN
+F 0 "#PWR018" H 3150 3400 50  0001 C CNN
 F 1 "GND" H 3150 3500 50  0000 C CNN
 F 2 "" H 3150 3650 50  0000 C CNN
@@
 $EndComp
 $Comp
-L GND #PWR018
+L GND #PWR019
 U 1 1 59D37473
 P 4750 3550
-F 0 "#PWR018" H 4750 3300 50  0001 C CNN
+F 0 "#PWR019" H 4750 3300 50  0001 C CNN
 F 1 "GND" H 4750 3400 50  0000 C CNN
 F 2 "" H 4750 3550 50  0000 C CNN
@@
 $EndComp
 $Comp
-L GND #PWR019
+L GND #PWR020
 U 1 1 59D39161
 P 5050 2750
-F 0 "#PWR019" H 5050 2500 50  0001 C CNN
+F 0 "#PWR020" H 5050 2500 50  0001 C CNN
 F 1 "GND" H 5050 2600 50  0000 C CNN
 F 2 "" H 5050 2750 50  0000 C CNN
@@
 $EndComp
 $Comp
-L GND #PWR020
+L GND #PWR021
 U 1 1 59D397E4
 P 4750 5550
-F 0 "#PWR020" H 4750 5300 50  0001 C CNN
+F 0 "#PWR021" H 4750 5300 50  0001 C CNN
 F 1 "GND" H 4750 5400 50  0000 C CNN
 F 2 "" H 4750 5550 50  0000 C CNN
@@
 $EndComp
 $Comp
-L +BATT #PWR021
+L +BATT #PWR022
 U 1 1 59D39851
 P 4750 4150
-F 0 "#PWR021" H 4750 4000 50  0001 C CNN
+F 0 "#PWR022" H 4750 4000 50  0001 C CNN
 F 1 "+BATT" H 4750 4290 50  0000 C CNN
 F 2 "" H 4750 4150 50  0000 C CNN
@@
 BATT_V_EN
 Wire Wire Line
-	6400 3100 6250 3100
-Wire Wire Line
-	6250 3100 6250 3000
+	6250 3100 6400 3100
+Wire Wire Line
+	6250 2850 6250 3100
 Connection ~ 6250 3000
 Wire Wire Line
@@
 F 0 "P1" H 2975 3075 50  0000 C CNN
 F 1 "USB_OTG" H 2650 3400 50  0000 C CNN
-F 2 "Connect:USB_Micro-B" V 2600 3100 50  0001 C CNN
+F 2 "Connectors_USB:USB_Micro-B_Molex_47346-0001" V 2600 3100 50  0001 C CNN
 F 3 "" V 2600 3100 50  0000 C CNN
 	1    2650 3200
@@
 	1    0    0    -1
 $EndComp
+$Comp
+L VBUS #PWR023
+U 1 1 59F894AA
+P 6250 2850
+F 0 "#PWR023" H 6250 2700 50  0001 C CNN
+F 1 "VBUS" H 6250 3000 50  0000 C CNN
+F 2 "" H 6250 2850 50  0001 C CNN
+F 3 "" H 6250 2850 50  0001 C CNN
+	1    6250 2850
+	1    0    0    -1
+$EndComp

Commit message: update board, schematics, add bmp280
Parts:
- P1: symbol USB_OTG -> USB_OTG-RESCUE-env_board
Changed lines of the file:
@@
 EESchema Schematic File Version 2
+LIBS:env_board-rescue
 LIBS:power
 LIBS:device
@@
 $EndComp
 $Comp
-L GND #PWR013
+L GND #PWR21
 U 1 1 59568C2C
 P 6700 3750
-F 0 "#PWR013" H 6700 3500 50  0001 C CNN
+F 0 "#PWR21" H 6700 3500 50  0001 C CNN
 F 1 "GND" H 6700 3600 50  0000 C CNN
 F 2 "" H 6700 3750 50  0000 C CNN
@@
 $EndComp
 $Comp
-L VDD #PWR014
+L VDD #PWR22
 U 1 1 59568C2F
 P 7100 2900
-F 0 "#PWR014" H 7100 2750 50  0001 C CNN
+F 0 "#PWR22" H 7100 2750 50  0001 C CNN
 F 1 "VDD" H 7100 3050 50  0000 C CNN
 F 2 "" H 7100 2900 50  0000 C CNN
@@
 $EndComp
 $Comp
-L GND #PWR015
+L GND #PWR14
 U 1 1 59568C3A
 P 3500 5100
-F 0 "#PWR015" H 3500 4850 50  0001 C CNN
+F 0 "#PWR14" H 3500 4850 50  0001 C CNN
 F 1 "GND" H 3500 4950 50  0000 C CNN
 F 2 "" H 3500 5100 50  0000 C CNN
@@
 $EndComp
 $Comp
-L +BATT #PWR016
+L +BATT #PWR13
 U 1 1 59568C5B
 P 3500 4900
-F 0 "#PWR016" H 3500 4750 50  0001 C CNN
+F 0 "#PWR13" H 3500 4750 50  0001 C CNN
 F 1 "+BATT" H 3500 5040 50  0000 C CNN
 F 2 "" H 3500 4900 50  0000 C CNN
@@
 Connection ~ 6700 3650
 $Comp
-L +BATT #PWR017
+L +BATT #PWR15
 U 1 1 5979B653
 P 4750 2900
-F 0 "#PWR017" H 4750 2750 50  0001 C CNN
+F 0 "#PWR15" H 4750 2750 50  0001 C CNN
 F 1 "+BATT" H 4750 3040 50  0000 C CNN
 F 2 "" H 4750 2900 50  0000 C CNN
@@
 $EndComp
 $Comp
-L GND #PWR018
+L GND #PWR12
 U 1 1 59D3742E
 P 3150 3650
-F 0 "#PWR018" H 3150 3400 50  0001 C CNN
+F 0 "#PWR12" H 3150 3400 50  0001 C CNN
 F 1 "GND" H 3150 3500 50  0000 C CNN
 F 2 "" H 3150 3650 50  0000 C CNN
@@
 $EndComp
 $Comp
-L GND #PWR019
+L GND #PWR16
 U 1 1 59D37473
 P 4750 3550
-F 0 "#PWR019" H 4750 3300 50  0001 C CNN
+F 0 "#PWR16" H 4750 3300 50  0001 C CNN
 F 1 "GND" H 4750 3400 50  0000 C CNN
 F 2 "" H 4750 3550 50  0000 C CNN
@@
 $EndComp
 $Comp
-L GND #PWR020
+L GND #PWR19
 U 1 1 59D39161
 P 5050 2750
-F 0 "#PWR020" H 5050 2500 50  0001 C CNN
+F 0 "#PWR19" H 5050 2500 50  0001 C CNN
 F 1 "GND" H 5050 2600 50  0000 C CNN
 F 2 "" H 5050 2750 50  0000 C CNN
@@
 $EndComp
 $Comp
-L GND #PWR021
+L GND #PWR18
 U 1 1 59D397E4
 P 4750 5550
-F 0 "#PWR021" H 4750 5300 50  0001 C CNN
+F 0 "#PWR18" H 4750 5300 50  0001 C CNN
 F 1 "GND" H 4750 5400 50  0000 C CNN
 F 2 "" H 4750 5550 50  0000 C CNN
@@
 $EndComp
 $Comp
-L +BATT #PWR022
+L +BATT #PWR17
 U 1 1 59D39851
 P 4750 4150
-F 0 "#PWR022" H 4750 4000 50  0001 C CNN
+F 0 "#PWR17" H 4750 4000 50  0001 C CNN
 F 1 "+BATT" H 4750 4290 50  0000 C CNN
 F 2 "" H 4750 4150 50  0000 C CNN
@@
 Connection ~ 3150 3550
 $Comp
-L USB_OTG P1
+L USB_OTG-RESCUE-env_board P1
 U 1 1 59DF246E
 P 2650 3200
+AR Path="/59DF246E" Ref="P1"  Part="1"
+AR Path="/596DCDC5/59DF246E" Ref="P1"  Part="1"
 F 0 "P1" H 2975 3075 50  0000 C CNN
 F 1 "USB_OTG" H 2650 3400 50  0000 C CNN
@@
 $EndComp
 $Comp
-L VBUS #PWR023
+L VBUS #PWR20
 U 1 1 59F894AA
 P 6250 2850
-F 0 "#PWR023" H 6250 2700 50  0001 C CNN
+F 0 "#PWR20" H 6250 2700 50  0001 C CNN
 F 1 "VBUS" H 6250 3000 50  0000 C CNN
 F 2 "" H 6250 2850 50  0001 C CNN

Commit message: update sensor and add housing for sensor
Parts:
- added D1: BAT20J, Diodes_SMD:SOD-323, symbol D_Schottky
- C5: value 2.2u -> 1u
- U4: value AP2204K-3.0 -> TLV74130
Connections:
- net VBUS: now also D2.2 (A), Q2.1 (G), R8.1, D1.1 (K); no longer C4.1, D2.1 (K), Q2.2 (S), U4.1 (VIN), U4.3 (EN)
- net at C2.1, P1.1 (VCC), U5.1 (CEN)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: now also D1.2 (A); no longer D2.2 (A), Q2.1 (G), R8.1
- new net: C4.1, D2.1 (K), Q2.2 (S), U4.1 (VIN), U4.3 (EN)
Changed lines of the file:
@@
 LIBS:rfcom
 LIBS:sensors
-LIBS:Battery_Management
 LIBS:env_board-cache
 EELAYER 25 0
@@
 P 7100 3350
 F 0 "C5" H 7125 3450 50  0000 L CNN
-F 1 "2.2u" H 7125 3250 50  0000 L CNN
+F 1 "1u" H 7125 3250 50  0000 L CNN
 F 2 "Capacitors_SMD:C_0603" H 7138 3200 50  0001 C CNN
 F 3 "" H 7100 3350 50  0000 C CNN
@@
 $EndComp
 $Comp
-L GND #PWR21
+L GND #PWR015
 U 1 1 59568C2C
 P 6700 3750
-F 0 "#PWR21" H 6700 3500 50  0001 C CNN
+F 0 "#PWR015" H 6700 3500 50  0001 C CNN
 F 1 "GND" H 6700 3600 50  0000 C CNN
 F 2 "" H 6700 3750 50  0000 C CNN
@@
 $EndComp
 $Comp
-L VDD #PWR22
+L VDD #PWR016
 U 1 1 59568C2F
 P 7100 2900
-F 0 "#PWR22" H 7100 2750 50  0001 C CNN
+F 0 "#PWR016" H 7100 2750 50  0001 C CNN
 F 1 "VDD" H 7100 3050 50  0000 C CNN
 F 2 "" H 7100 2900 50  0000 C CNN
@@
 $EndComp
 $Comp
-L GND #PWR14
+L GND #PWR017
 U 1 1 59568C3A
 P 3500 5100
-F 0 "#PWR14" H 3500 4850 50  0001 C CNN
+F 0 "#PWR017" H 3500 4850 50  0001 C CNN
 F 1 "GND" H 3500 4950 50  0000 C CNN
 F 2 "" H 3500 5100 50  0000 C CNN
@@
 $EndComp
 $Comp
-L +BATT #PWR13
+L +BATT #PWR018
 U 1 1 59568C5B
 P 3500 4900
-F 0 "#PWR13" H 3500 4750 50  0001 C CNN
+F 0 "#PWR018" H 3500 4750 50  0001 C CNN
 F 1 "+BATT" H 3500 5040 50  0000 C CNN
 F 2 "" H 3500 4900 50  0000 C CNN
@@
 Connection ~ 6700 3650
 $Comp
-L +BATT #PWR15
+L +BATT #PWR019
 U 1 1 5979B653
 P 4750 2900
-F 0 "#PWR15" H 4750 2750 50  0001 C CNN
+F 0 "#PWR019" H 4750 2750 50  0001 C CNN
 F 1 "+BATT" H 4750 3040 50  0000 C CNN
 F 2 "" H 4750 2900 50  0000 C CNN
@@
 $EndComp
 $Comp
-L GND #PWR12
+L GND #PWR020
 U 1 1 59D3742E
 P 3150 3650
-F 0 "#PWR12" H 3150 3400 50  0001 C CNN
+F 0 "#PWR020" H 3150 3400 50  0001 C CNN
 F 1 "GND" H 3150 3500 50  0000 C CNN
 F 2 "" H 3150 3650 50  0000 C CNN
@@
 $EndComp
 $Comp
-L GND #PWR16
+L GND #PWR021
 U 1 1 59D37473
 P 4750 3550
-F 0 "#PWR16" H 4750 3300 50  0001 C CNN
+F 0 "#PWR021" H 4750 3300 50  0001 C CNN
 F 1 "GND" H 4750 3400 50  0000 C CNN
 F 2 "" H 4750 3550 50  0000 C CNN
@@
 P 6700 3100
 F 0 "U4" H 6500 3325 50  0000 L CNN
-F 1 "AP2204K-3.0" H 6700 3325 50  0000 L CNN
+F 1 "TLV74130" H 6700 3325 50  0000 L CNN
 F 2 "TO_SOT_Packages_SMD:SOT-23-5" H 6700 3425 50  0001 C CNN
 F 3 "" H 6700 3200 50  0001 C CNN
@@
 $EndComp
 $Comp
-L GND #PWR19
+L GND #PWR022
 U 1 1 59D39161
 P 5050 2750
-F 0 "#PWR19" H 5050 2500 50  0001 C CNN
+F 0 "#PWR022" H 5050 2500 50  0001 C CNN
 F 1 "GND" H 5050 2600 50  0000 C CNN
 F 2 "" H 5050 2750 50  0000 C CNN
@@
 	5400 2600 5800 2600
 Wire Wire Line
-	5500 2400 5500 2700
+	5500 2300 5500 2700
 $Comp
 L D_Schottky D2
@@
 	5800 2600 5800 2650
 Connection ~ 5500 2600
-Wire Wire Line
-	3450 2400 5500 2400
 $Comp
 L R R2
@@
 $EndComp
 $Comp
-L GND #PWR18
+L GND #PWR023
 U 1 1 59D397E4
 P 4750 5550
-F 0 "#PWR18" H 4750 5300 50  0001 C CNN
+F 0 "#PWR023" H 4750 5300 50  0001 C CNN
 F 1 "GND" H 4750 5400 50  0000 C CNN
 F 2 "" H 4750 5550 50  0000 C CNN
@@
 $EndComp
 $Comp
-L +BATT #PWR17
+L +BATT #PWR024
 U 1 1 59D39851
 P 4750 4150
-F 0 "#PWR17" H 4750 4000 50  0001 C CNN
+F 0 "#PWR024" H 4750 4000 50  0001 C CNN
 F 1 "+BATT" H 4750 4290 50  0000 C CNN
 F 2 "" H 4750 4150 50  0000 C CNN
@@
 Wire Wire Line
 	6250 3100 6400 3100
-Wire Wire Line
-	6250 2850 6250 3100
 Connection ~ 6250 3000
 Wire Wire Line
@@
 $EndComp
 $Comp
-L VBUS #PWR20
+L VBUS #PWR025
 U 1 1 59F894AA
-P 6250 2850
-F 0 "#PWR20" H 6250 2700 50  0001 C CNN
-F 1 "VBUS" H 6250 3000 50  0000 C CNN
-F 2 "" H 6250 2850 50  0001 C CNN
-F 3 "" H 6250 2850 50  0001 C CNN
-	1    6250 2850
-	1    0    0    -1
-$EndComp
+P 5500 2300
+F 0 "#PWR025" H 5500 2150 50  0001 C CNN
+F 1 "VBUS" H 5500 2450 50  0000 C CNN
+F 2 "" H 5500 2300 50  0001 C CNN
+F 3 "" H 5500 2300 50  0001 C CNN
+	1    5500 2300
+	1    0    0    -1
+$EndComp
+Connection ~ 5500 2400
+Wire Wire Line
+	6250 3100 6250 3000
+$Comp
+L D_Schottky D1
+U 1 1 5A8FF863
+P 4800 2400
+F 0 "D1" H 4800 2500 50  0000 C CNN
+F 1 "BAT20J" H 4800 2300 50  0000 C CNN
+F 2 "Diodes_SMD:SOD-323" H 4800 2400 50  0001 C CNN
+F 3 "" H 4800 2400 50  0001 C CNN
+	1    4800 2400
+	-1   0    0    1
+$EndComp
+Wire Wire Line
+	3450 2400 4650 2400
+Wire Wire Line
+	4950 2400 5500 2400
 $EndSCHEMATC

Commit message: update sensor/housings
Parts:
- added Q3: DMP3099L-13, Package_TO_SOT_SMD:SOT-23, symbol Device:Q_PMOS_GSD
- added R5: 10k, Resistor_SMD:R_0603_1608Metric, symbol Device:R
- C2, C3, C4, C5: footprint Capacitors_SMD:C_0603 -> Capacitor_SMD:C_0603_1608Metric; symbol C -> Device:C
- D1, D2: footprint Diodes_SMD:SOD-323 -> Diode_SMD:D_SOD-323; symbol D_Schottky -> Device:D_Schottky
- J2: footprint Connectors_JST:JST_PH_S2B-PH-K_02x2.00mm_Angled -> Connector_JST:JST_PH_S2B-PH-K_1x02_P2.00mm_Horizontal; symbol CONN_01X02 -> Connector_Generic:Conn_01x02
- P1: footprint Connectors_USB:USB_Micro-B_Molex_47346-0001 -> Connector_USB:USB_Micro-B_Molex_47346-0001; symbol USB_OTG-RESCUE-env_board -> Connector_Specialized:USB_B_Micro
- Q1: value Q_NMOS_GSD -> NX7002AKVL; footprint TO_SOT_Packages_SMD:SOT-23 -> Package_TO_SOT_SMD:SOT-23; symbol Q_NMOS_GSD -> Device:Q_NMOS_GSD
- Q2: value Q_PMOS_GSD -> DMP3099L-13; footprint TO_SOT_Packages_SMD:SOT-23 -> Package_TO_SOT_SMD:SOT-23; symbol Q_PMOS_GSD -> Device:Q_PMOS_GSD
- R2, R7, R8: footprint Resistors_SMD:R_0603 -> Resistor_SMD:R_0603_1608Metric; symbol R -> Device:R
- U4: footprint TO_SOT_Packages_SMD:SOT-23-5 -> Package_TO_SOT_SMD:SOT-23-5; symbol AP2204K-3.0 -> Regulator_Linear:AP2204K-3.0
- U5: footprint TO_SOT_Packages_SMD:SOT-23-5 -> Package_TO_SOT_SMD:SOT-23-5; symbol MCP73811T-420I-OT -> Battery_Management:MCP73811T-420I-OT
Connections:
- wire segments 41 -> 66
Other:
- moved on the sheet: Q1, R2, R7
